Commit message: updated xacro macros to handle new effort control mode

File: kortex_description/arms/gen3/7dof/urdf/gen3_macro.xacro (robot description, xacro)
@@ -29,5 +29,7 @@
     isaac_joint_states:=/isaac_joint_states
     use_external_cable:=false
-    initial_positions:=${dict(joint_1=0.0,joint_2=0.0,joint_3=0.0,joint_4=0.0,joint_5=0.0,joint_6=0.0,joint_7=0.0)}" >
+    initial_positions:=${dict(joint_1=0.0,joint_2=0.0,joint_3=0.0,joint_4=0.0,joint_5=0.0,joint_6=0.0,joint_7=0.0)}
+    high_velocity_torque_mode:=false
+    gravity_compensation_urdf:=${find kortex_description}/robots/gen3_7dof_2f85_intertial.urdf" >
     <!-- ros2 control include -->
     <xacro:include filename="$(find kortex_description)/arms/gen3/${dof}dof/urdf/kortex.ros2_control.xacro" />
@@ -53,5 +55,7 @@
       gripper_max_velocity="${gripper_max_velocity}"
       gripper_max_force="${gripper_max_force}"
-      gripper_joint_name="${gripper_joint_name}"/>
+      gripper_joint_name="${gripper_joint_name}"
+      high_velocity_torque_mode="${high_velocity_torque_mode}"
+      gravity_compensation_urdf:="${gravity_compensation_urdf}"/>
     <joint name="${prefix}base_joint" type="fixed">
       <xacro:insert_block name="origin" />
@@ -77,5 +81,5 @@
         <origin xyz="0 0 0" rpy="0 0 0" />
         <geometry>
-          <mesh filename="file://$(find kortex_description)/arms/gen3/${dof}dof/meshes/base_link.dae" />
+          <mesh filename="file://$(find kortex_description)/arms/gen3/${dof}dof/meshes/collision/base_link.STL" />
         </geometry>
       </collision>
@@ -99,5 +103,5 @@
         <origin xyz="0 0 0" rpy="0 0 0" />
         <geometry>
-          <mesh filename="file://$(find kortex_description)/arms/gen3/${dof}dof/meshes/shoulder_link.dae" />
+          <mesh filename="file://$(find kortex_description)/arms/gen3/${dof}dof/meshes/collision/shoulder_link.STL" />
         </geometry>
       </collision>
@@ -155,5 +159,5 @@
         <origin xyz="0 0 0" rpy="0 0 0" />
         <geometry>
-          <mesh filename="file://$(find kortex_description)/arms/gen3/${dof}dof/meshes/half_arm_1_link.dae" />
+          <mesh filename="file://$(find kortex_description)/arms/gen3/${dof}dof/meshes/collision/half_arm_1_link.STL" />
         </geometry>
       </collision>
@@ -189,5 +193,5 @@
         <origin xyz="0 0 0" rpy="0 0 0" />
         <geometry>
-          <mesh filename="file://$(find kortex_description)/arms/gen3/${dof}dof/meshes/half_arm_2_link.dae" />
+          <mesh filename="file://$(find kortex_description)/arms/gen3/${dof}dof/meshes/collision/half_arm_2_link.STL" />
         </geometry>
       </collision>
@@ -245,5 +249,5 @@
         <origin xyz="0 0 0" rpy="0 0 0" />
         <geometry>
-          <mesh filename="file://$(find kortex_description)/arms/gen3/${dof}dof/meshes/forearm_link.dae" />
+          <mesh filename="file://$(find kortex_description)/arms/gen3/${dof}dof/meshes/collision/forearm_link.STL" />
         </geometry>
       </collision>
@@ -279,5 +283,5 @@
         <origin xyz="0 0 0" rpy="0 0 0" />
         <geometry>
-          <mesh filename="file://$(find kortex_description)/arms/gen3/${dof}dof/meshes/spherical_wrist_1_link.dae" />
+          <mesh filename="file://$(find kortex_description)/arms/gen3/${dof}dof/meshes/collision/spherical_wrist_1_link.STL" />
         </geometry>
       </collision>
@@ -335,5 +339,5 @@
         <origin xyz="0 0 0" rpy="0 0 0" />
         <geometry>
-          <mesh filename="file://$(find kortex_description)/arms/gen3/${dof}dof/meshes/spherical_wrist_2_link.dae" />
+          <mesh filename="file://$(find kortex_description)/arms/gen3/${dof}dof/meshes/collision/spherical_wrist_2_link.STL" />
         </geometry>
       </collision>
@@ -370,5 +374,5 @@
         <origin xyz="0 0 0" rpy="0 0 0" />
         <geometry>
-          <mesh filename="file://$(find kortex_description)/arms/gen3/${dof}dof/meshes/bracelet_with_vision_link.dae" />
+          <mesh filename="file://$(find kortex_description)/arms/gen3/${dof}dof/meshes/collision/bracelet_with_vision_link.STL" />
         </geometry>
       </collision>
@@ -394,5 +398,5 @@
         <origin xyz="0 0 0" rpy="0 0 0" />
         <geometry>
-          <mesh filename="file://$(find kortex_description)/arms/gen3/${dof}dof/meshes/bracelet_no_vision_link.dae" />
+          <mesh filename="file://$(find kortex_description)/arms/gen3/${dof}dof/meshes/collision/bracelet_no_vision_link.STL" />
         </geometry>
       </collision>

File: kortex_description/arms/gen3/7dof/urdf/kortex.ros2_control.xacro (robot description, xacro)
@@ -23,5 +23,7 @@
     gripper_joint_name
     gripper_max_velocity:=100.0
-    gripper_max_force:=100.0">
+    gripper_max_force:=100.0
+    high_velocity_torque_mode:=false
+    gravity_compensation_urdf:=${find kortex_description}/robots/gen3_7dof_2f85_intertial.urdf">
     <ros2_control name="${name}" type="system">
       <hardware>
@@ -56,10 +58,14 @@
           <param name="gripper_max_velocity">${gripper_max_velocity}</param>
           <param name="gripper_max_force">${gripper_max_force}</param>
+          <param name="high_velocity_torque_mode">${high_velocity_torque_mode}</param>
+          <param name="gravity_compensation_urdf">${gravity_compensation_urdf}</param>
         </xacro:unless>
       </hardware>
       <joint name="${prefix}joint_1">
+        <command_interface name="effort"/>
+        <command_interface name="velocity"/>
         <command_interface name="position">
-          <param name="min">{-2*pi}</param>
-          <param name="max">{2*pi}</param>
+          <param name="min">${-2*pi}</param>
+          <param name="max">${2*pi}</param>
         </command_interface>
         <state_interface name="position">
@@ -70,4 +76,6 @@
       </joint>
       <joint name="${prefix}joint_2">
+        <command_interface name="effort"/>
+        <command_interface name="velocity"/>
         <command_interface name="position">
           <param name="min">-2.41</param>
@@ -81,7 +89,9 @@
       </joint>
       <joint name="${prefix}joint_3">
+        <command_interface name="effort"/>
+        <command_interface name="velocity"/>
         <command_interface name="position">
-          <param name="min">{-2*pi}</param>
-          <param name="max">{2*pi}</param>
+          <param name="min">${-2*pi}</param>
+          <param name="max">${2*pi}</param>
         </command_interface>
         <state_interface name="position">
@@ -92,4 +102,6 @@
       </joint>
       <joint name="${prefix}joint_4">
+        <command_interface name="effort"/>
+        <command_interface name="velocity"/>
         <command_interface name="position">
           <param name="min">-2.66</param>
@@ -103,7 +115,9 @@
       </joint>
       <joint name="${prefix}joint_5">
+        <command_interface name="effort"/>
+        <command_interface name="velocity"/>
         <command_interface name="position">
-          <param name="min">{-2*pi}</param>
-          <param name="max">{2*pi}</param>
+          <param name="min">${-2*pi}</param>
+          <param name="max">${2*pi}</param>
         </command_interface>
         <state_interface name="position">
@@ -114,4 +128,6 @@
       </joint>
       <joint name="${prefix}joint_6">
+        <command_interface name="effort"/>
+        <command_interface name="velocity"/>
         <command_interface name="position">
           <param name="min">-2.23</param>
@@ -125,7 +141,9 @@
       </joint>
       <joint name="${prefix}joint_7">
+        <command_interface name="effort"/>
+        <command_interface name="velocity"/>
         <command_interface name="position">
-          <param name="min">{-2*pi}</param>
-          <param name="max">{2*pi}</param>
+          <param name="min">${-2*pi}</param>
+          <param name="max">${2*pi}</param>
         </command_interface>
         <state_interface name="position">
@@ -139,4 +157,5 @@
           <joint name="${prefix}${gripper_joint_name}">
             <command_interface name="position" />
+            <command_interface name="velocity"/>
             <state_interface name="position"/>
             <state_interface name="velocity"/>

File: kortex_description/grippers/robotiq_2f_85/urdf/robotiq_2f_85_macro.xacro (robot description, xacro)
@@ -27,7 +27,5 @@
         fake_sensor_commands="${fake_sensor_commands}"
         sim_ignition="${sim_ignition}"
-        sim_isaac="${sim_isaac}"
-        isaac_joint_commands="${isaac_joint_commands}"
-        isaac_joint_states="${isaac_joint_states}">
+        sim_isaac="${sim_isaac}">
         <origin xyz="0 0 0" rpy="0 0 0" />
     </xacro:robotiq_gripper>

File: kortex_description/robots/gen3_7dof_2f85_inertial.urdf (robot description, URDF)
Before this commit: robot gen3_, 31 links, 30 joints
Links:
- removed link world
- removed link wrist_mounted_camera_color_frame
- removed link wrist_mounted_camera_color_optical_frame
- removed link wrist_mounted_camera_depth_frame
- removed link wrist_mounted_camera_depth_optical_frame
- removed link wrist_mounted_camera_infra1_frame
- removed link wrist_mounted_camera_infra1_optical_frame
- removed link wrist_mounted_camera_infra2_frame
- removed link wrist_mounted_camera_infra2_optical_frame
- link wrist_camera_mount_link: mass 0.5 -> None
- link wrist_mounted_camera_link: mass 0.072 -> None
Joints:
- removed joint gen3_base_joint
- removed joint wrist_mounted_camera_color_joint
- removed joint wrist_mounted_camera_color_optical_joint
- removed joint wrist_mounted_camera_depth_joint
- removed joint wrist_mounted_camera_depth_optical_joint
- removed joint wrist_mounted_camera_infra1_joint
- removed joint wrist_mounted_camera_infra1_optical_joint
- removed joint wrist_mounted_camera_infra2_joint
- removed joint wrist_mounted_camera_infra2_optical_joint
- joint gen3_robotiq_85_left_finger_tip_joint: type continuous -> fixed
- joint gen3_robotiq_85_left_inner_knuckle_joint: type continuous -> fixed
- joint gen3_robotiq_85_left_knuckle_joint: type revolute -> fixed
- joint gen3_robotiq_85_right_finger_tip_joint: type continuous -> fixed
- joint gen3_robotiq_85_right_inner_knuckle_joint: type continuous -> fixed
- joint gen3_robotiq_85_right_knuckle_joint: type revolute -> fixed
